File: hardware/board/board.kicad_pcb (KiCad board)
At the start: 2 copper layers, 100 x 30 mm, 55 parts, among them J1 DC THRU, J2 DC THRU, J3 DC OUT, J4 DC IN, J5 DC IN, J6 DC OUT, J7 Eurorack Power, J8 Eurorack Power, SW1 ON/OFF, U1 VX7805-500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

Commit message: remove Winterbloom logo in order to conform to license add JLCPCB production files
Parts:
- removed WNTR: LOGO, LOGO
